File: hardware/devboard.kicad_sch (KiCad schematic)
At the start: 8 parts, among them J1 Barrel_Jack_12V, J2 5V_OUT_TO_FPGA, J3 3V3_OUT_TO_UART, U1 REG_5V0, U2 REG_3V3

Commit message: Demo: introduce duplicate reference designator (C2 -> C1)
Deliberately broken branch to exercise the erc job in kicad-ci.yml.
C2 (output cap on the 5V rail) now shares its reference with the
existing C1 (input cap) -- kicad-cli sch erc should flag this as a
duplicate reference error and fail the erc job, while spice-verify
still passes since the electrical values are untouched.

Co-Authored-By: Claude Sonnet 5 <noreply@anthropic.com>
Parts:
- renumbered C2 to C1
Changed lines of the file:
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@@
 	(symbol (lib_id "utoss:CAP") (at 60 20 0) (unit 1)
 		(in_bom yes) (on_board yes) (dnp no)
-		(property "Reference" "C2" (at 60 23.81 0) (effects (font (size 1.27 1.27))))
+		(property "Reference" "C1" (at 60 23.81 0) (effects (font (size 1.27 1.27))))
 		(property "Value" "22uF_Cout5V" (at 60 16.19 0) (effects (font (size 1.27 1.27))))
 		(property "Footprint" "" (at 60 20 0) (effects (font (size 1.27 1.27)) hide))
 		(property "Datasheet" "" (at 60 20 0) (effects (font (size 1.27 1.27)) hide))
-		(instances (project "devboard" (path "/00000000-0000-0000-0000-000000000000" (reference "C2") (unit 1))))
+		(instances (project "devboard" (path "/00000000-0000-0000-0000-000000000000" (reference "C1") (unit 1))))
 	)
 	(symbol (lib_id "utoss:CONN2") (at 80 20 0) (unit 1)
