File: hardware/devboard.kicad_sch (KiCad schematic)
At the start: 8 parts, among them J1 Barrel_Jack_12V, J2 5V_OUT_TO_FPGA, J3 3V3_OUT_TO_UART, U1 REG_5V0, U2 REG_3V3

Commit message: Demo: legitimate in-spec change (bump input cap 10uF -> 22uF)
Passing-case counterpart to demo/power-fail-erc and demo/power-fail-spec:
a real, harmless design tweak that should sail through both erc and
spice-verify unchanged.

Co-Authored-By: Claude Sonnet 5 <noreply@anthropic.com>
Parts:
- C1: value 10uF_Cin -> 22uF_Cin
Changed lines of the file:
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@@
 		(in_bom yes) (on_board yes) (dnp no)
 		(property "Reference" "C1" (at 20 23.81 0) (effects (font (size 1.27 1.27))))
-		(property "Value" "10uF_Cin" (at 20 16.19 0) (effects (font (size 1.27 1.27))))
+		(property "Value" "22uF_Cin" (at 20 16.19 0) (effects (font (size 1.27 1.27))))
 		(property "Footprint" "" (at 20 20 0) (effects (font (size 1.27 1.27)) hide))
 		(property "Datasheet" "" (at 20 20 0) (effects (font (size 1.27 1.27)) hide))
